Commit message: added scan to scan

File: rmcl_sim/urdf/ceres.urdf.xacro (robot description, xacro)
@@ -118,4 +118,30 @@
     <origin xyz="0 0 ${body_height/2 + 0.4}"/>
   </joint>
+  <link name="sick_tim">
+    <visual>
+      <origin xyz="0 0 0" rpy="0 0 0" />
+      <geometry>
+        <cylinder radius="0.05" length="0.05"/>
+      </geometry>
+      <material name="blue" >
+        <color rgba="0 0 1 1" />
+      </material>
+    </visual>
+    <collision>
+      <geometry>
+        <cylinder radius="0.05" length="0.1"/>
+      </geometry>
+    </collision>
+     <xacro:cylinder_inertial
+      radius="0.05"
+      length="0.1"
+      mass="0.1"
+      />
+  </link>
+  <joint name="sick_tim_to_base_joint" type="fixed">
+    <parent link="base_link" />
+    <child link="sick_tim" />
+    <origin xyz="0 0 ${body_height/2 + 0.2}"/>
+  </joint>
   <!-- Gazebo Plugins -->
   <gazebo reference="imu" >
@@ -131,5 +157,5 @@
   </gazebo>
   <gazebo reference="velodyne">
-    <sensor name="velodyne-vlp16" type='gpu_lidar'>"
+    <sensor name="velodyne-vlp16" type="gpu_lidar">
       <pose relative_to="velodyne">0 0 0 0 0 0</pose>
       <topic>/model/robot/cloud</topic>
@@ -163,4 +189,37 @@
     </sensor>
   </gazebo>
+  <gazebo reference="sick_tim">
+    <sensor name="sick_tim" type="gpu_lidar">
+      <pose relative_to="sick_tim">0 0 0 0 0 0</pose>
+      <topic>/model/robot/scan</topic>
+      <update_rate>10</update_rate>
+      <ray>
+        <scan>
+          <horizontal>
+            <samples>270</samples>
+            <resolution>1</resolution>
+            <min_angle>-${M_PI*3.0/4.0}</min_angle>
+            <max_angle>${M_PI*3.0/4.0}</max_angle>
+          </horizontal>
+          <vertical>
+            <samples>1</samples>
+            <resolution>0.01</resolution>
+            <min_angle>0</min_angle>
+            <max_angle>0</max_angle>
+          </vertical>
+        </scan>
+        <range>
+          <min>0.08</min>
+          <max>20.0</max>
+          <resolution>0.01</resolution>
+        </range>
+      </ray>
+      <always_on>1</always_on>
+      <visualize>true</visualize>
+      <frame_id>velodyne</frame_id>
+      <gz_frame_id>velodyne</gz_frame_id>
+      <ign_frame_id>velodyne</ign_frame_id>
+    </sensor>
+  </gazebo>
   <gazebo>
     <plugin

Commit message: added flags to enable different sensors

File: rmcl_sim/urdf/ceres.urdf.xacro (robot description, xacro)
@@ -8,4 +8,8 @@
   <xacro:include filename="$(find rmcl_sim)/urdf/common.urdf.xacro" />
   <xacro:include filename="$(find rmcl_sim)/urdf/wheel.urdf.xacro" />
+  <!-- Args -->
+  <xacro:arg name="velodyne_vlp16" default="true"/>
+  <xacro:arg name="sick_tim" default="false"/>
+  <xacro:arg name="asus_xtion" default="false"/>
   <xacro:property name="M_PI" value="3.14159265359"/>
   <xacro:property name="imu_stdev" value="0.0001" />
@@ -92,56 +96,4 @@
     <origin xyz="${imu_offset_x} ${imu_offset_y} ${imu_offset_z}" rpy="${M_PI} 0 ${M_PI/2.0}" />
   </joint>
-  <link name="velodyne">
-    <visual>
-      <origin xyz="0 0 0" rpy="0 0 0" />
-      <geometry>
-        <cylinder radius="0.05" length="0.1"/>
-      </geometry>
-      <material name="red" >
-        <color rgba="1 0 0 1" />
-      </material>
-    </visual>
-    <collision>
-      <geometry>
-        <cylinder radius="0.05" length="0.1"/>
-      </geometry>
-    </collision>
-     <xacro:cylinder_inertial
-      radius="0.05"
-      length="0.1"
-      mass="0.1"
-      />
-  </link>
-  <joint name="velodyne_to_base_joint" type="fixed">
-    <parent link="base_link" />
-    <child link="velodyne" />
-    <origin xyz="0 0 ${body_height/2 + 0.4}"/>
-  </joint>
-  <link name="sick_tim">
-    <visual>
-      <origin xyz="0 0 0" rpy="0 0 0" />
-      <geometry>
-        <cylinder radius="0.05" length="0.05"/>
-      </geometry>
-      <material name="blue" >
-        <color rgba="0 0 1 1" />
-      </material>
-    </visual>
-    <collision>
-      <geometry>
-        <cylinder radius="0.05" length="0.1"/>
-      </geometry>
-    </collision>
-     <xacro:cylinder_inertial
-      radius="0.05"
-      length="0.1"
-      mass="0.1"
-      />
-  </link>
-  <joint name="sick_tim_to_base_joint" type="fixed">
-    <parent link="base_link" />
-    <child link="sick_tim" />
-    <origin xyz="0 0 ${body_height/2 + 0.2}"/>
-  </joint>
   <!-- Gazebo Plugins -->
   <gazebo reference="imu" >
@@ -156,70 +108,178 @@
     </sensor>
   </gazebo>
-  <gazebo reference="velodyne">
-    <sensor name="velodyne-vlp16" type="gpu_lidar">
-      <pose relative_to="velodyne">0 0 0 0 0 0</pose>
-      <topic>/model/robot/cloud</topic>
-      <update_rate>10</update_rate>
-      <ray>
-        <scan>
-          <horizontal>
-            <samples>440</samples>
-            <resolution>1</resolution>
-            <min_angle>${-M_PI}</min_angle>
-            <max_angle>${M_PI}</max_angle>
-          </horizontal>
-          <vertical>
-            <samples>16</samples>
+  <xacro:if value="$(arg velodyne_vlp16)">
+    <link name="velodyne">
+      <visual>
+        <origin xyz="0 0 0" rpy="0 0 0" />
+        <geometry>
+          <cylinder radius="0.05" length="0.1"/>
+        </geometry>
+        <material name="red" >
+          <color rgba="1 0 0 1" />
+        </material>
+      </visual>
+      <collision>
+        <geometry>
+          <cylinder radius="0.05" length="0.1"/>
+        </geometry>
+      </collision>
+      <xacro:cylinder_inertial
+        radius="0.05"
+        length="0.1"
+        mass="0.1"
+        />
+    </link>
+    <joint name="velodyne_to_base_joint" type="fixed">
+      <parent link="base_link" />
+      <child link="velodyne" />
+      <origin xyz="0 0 ${body_height/2 + 0.4}"/>
+    </joint>
+    <gazebo reference="velodyne">
+      <sensor name="velodyne" type="gpu_lidar">
+        <pose relative_to="velodyne">0 0 0 0 0 0</pose>
+        <topic>/model/robot/cloud</topic>
+        <update_rate>10</update_rate>
+        <ray>
+          <scan>
+            <horizontal>
+              <samples>440</samples>
+              <resolution>1</resolution>
+              <min_angle>${-M_PI}</min_angle>
+              <max_angle>${M_PI}</max_angle>
+            </horizontal>
+            <vertical>
+              <samples>16</samples>
+              <resolution>0.01</resolution>
+              <min_angle>-${M_PI*15.0/180.0}</min_angle>
+              <max_angle> ${M_PI*15.0/180.0}</max_angle>
+            </vertical>
+          </scan>
+          <range>
+            <min>0.2</min>
+            <max>100.0</max>
             <resolution>0.01</resolution>
-            <min_angle>-${M_PI*15.0/180.0}</min_angle>
-            <max_angle> ${M_PI*15.0/180.0}</max_angle>
-          </vertical>
-        </scan>
-        <range>
-          <min>0.2</min>
-          <max>100.0</max>
-          <resolution>0.01</resolution>
-        </range>
-      </ray>
-      <always_on>1</always_on>
-      <visualize>true</visualize>
-      <frame_id>velodyne</frame_id>
-      <gz_frame_id>velodyne</gz_frame_id>
-      <ign_frame_id>velodyne</ign_frame_id>
-    </sensor>
-  </gazebo>
-  <gazebo reference="sick_tim">
-    <sensor name="sick_tim" type="gpu_lidar">
-      <pose relative_to="sick_tim">0 0 0 0 0 0</pose>
-      <topic>/model/robot/scan</topic>
-      <update_rate>10</update_rate>
-      <ray>
-        <scan>
-          <horizontal>
-            <samples>270</samples>
-            <resolution>1</resolution>
-            <min_angle>-${M_PI*3.0/4.0}</min_angle>
-            <max_angle>${M_PI*3.0/4.0}</max_angle>
-          </horizontal>
-          <vertical>
-            <samples>1</samples>
+          </range>
+        </ray>
+        <always_on>1</always_on>
+        <visualize>true</visualize>
+        <frame_id>velodyne</frame_id>
+        <gz_frame_id>velodyne</gz_frame_id>
+        <ign_frame_id>velodyne</ign_frame_id>
+      </sensor>
+    </gazebo>
+  </xacro:if>
+  <xacro:if value="$(arg sick_tim)">
+    <link name="sick_tim">
+      <visual>
+        <origin xyz="0 0 0" rpy="0 0 0" />
+        <geometry>
+          <cylinder radius="0.05" length="0.05"/>
+        </geometry>
+        <material name="blue" >
+          <color rgba="0 0 1 1" />
+        </material>
+      </visual>
+      <collision>
+        <geometry>
+          <cylinder radius="0.05" length="0.1"/>
+        </geometry>
+      </collision>
+      <xacro:cylinder_inertial
+        radius="0.05"
+        length="0.1"
+        mass="0.1"
+        />
+    </link>
+    <joint name="sick_tim_to_base_joint" type="fixed">
+      <parent link="base_link" />
+      <child link="sick_tim" />
+      <origin xyz="0 0 ${body_height/2 + 0.2}"/>
+    </joint>
+    <gazebo reference="sick_tim">
+      <sensor name="sick_tim" type="gpu_lidar">
+        <pose relative_to="sick_tim">0 0 0 0 0 0</pose>
+        <topic>/model/robot/scan</topic>
+        <update_rate>10</update_rate>
+        <ray>
+          <scan>
+            <horizontal>
+              <samples>270</samples>
+              <resolution>1</resolution>
+              <min_angle>-${M_PI*3.0/4.0}</min_angle>
+              <max_angle>${M_PI*3.0/4.0}</max_angle>
+            </horizontal>
+            <vertical>
+              <samples>1</samples>
+              <resolution>0.01</resolution>
+              <min_angle>0</min_angle>
+              <max_angle>0</max_angle>
+            </vertical>
+          </scan>
+          <range>
+            <min>0.08</min>
+            <max>20.0</max>
             <resolution>0.01</resolution>
-            <min_angle>0</min_angle>
-            <max_angle>0</max_angle>
-          </vertical>
-        </scan>
-        <range>
-          <min>0.08</min>
-          <max>20.0</max>
-          <resolution>0.01</resolution>
-        </range>
-      </ray>
-      <always_on>1</always_on>
-      <visualize>true</visualize>
-      <frame_id>velodyne</frame_id>
-      <gz_frame_id>velodyne</gz_frame_id>
-      <ign_frame_id>velodyne</ign_frame_id>
-    </sensor>
-  </gazebo>
+          </range>
+        </ray>
+        <always_on>1</always_on>
+        <visualize>true</visualize>
+        <frame_id>velodyne</frame_id>
+        <gz_frame_id>velodyne</gz_frame_id>
+        <ign_frame_id>velodyne</ign_frame_id>
+      </sensor>
+    </gazebo>
+  </xacro:if>
+  <xacro:if value="$(arg asus_xtion)">
+    <link name="asus_xtion">
+      <visual>
+        <origin xyz="0 0 0" rpy="0 0 0" />
+        <geometry>
+          <box size="0.03 0.1 0.05"/>
+        </geometry>
+        <material name="green" >
+          <color rgba="0 1 0 1" />
+        </material>
+      </visual>
+      <collision>
+        <geometry>
+          <box size="0.03 0.1 0.05" />
+        </geometry>
+      </collision>
+      <xacro:box_inertial
+        x="0.03"
+        y="0.1"
+        z="0.05"
+        mass="0.1"
+        />
+    </link>
+    <joint name="asus_xtion_to_base_joint" type="fixed">
+      <parent link="base_link" />
+      <child link="asus_xtion" />
+      <origin xyz="0.2 0 ${body_height/2 + 0.1}" rpy="0.0 0.2 0.0" />
+    </joint>
+    <gazebo reference="asus_xtion">
+      <sensor name="asus_xtion" type="rgbd_camera">
+        <camera>
+          <horizontal_fov>1.047</horizontal_fov>
+          <image>
+            <width>320</width>
+            <height>240</height>
+          </image>
+          <clip>
+            <near>0.1</near>
+            <far>100</far>
+          </clip>
+        </camera>
+        <always_on>1</always_on>
+        <update_rate>30</update_rate>
+        <visualize>true</visualize>
+        <topic>/model/robot/rgbd_camera</topic>
+        <enable_metrics>true</enable_metrics>
+        <frame_id>asus_xtion</frame_id>
+        <gz_frame_id>asus_xtion</gz_frame_id>
+        <ign_frame_id>asus_xtion</ign_frame_id>
+      </sensor>
+    </gazebo>
+  </xacro:if>
   <gazebo>
     <plugin
